File: Dazzler.kicad_pcb (KiCad board)
At the start: 2 copper layers, 254 x 134.6 mm, 67 parts, among them J1 DIP-pad, J2 DIP-pad, J3 DIP-pad, J4 DIP-pad, J5 DIP-pad, J6 DIP-pad, J7 DIP-pad, P1 S100_MALE

Commit message: Add files via upload
Parts:
- removed 3408, 7402, 7405 (x3), 7495, 74LS08, 74LS10, 74LS30, 74LS32: DIP-14_W7.62mm_vintage, Dazzler:DIP-14_W7.62mm_vintage
- removed the 7404 at (174.9, 45.6)
- removed the 7404 at (83.2, 70.8)
- removed the 7404 at (106.3, 45.6)
- removed the 7408 at (83.4, 45.6)
- removed the 74175 at (245.1, 45.8)
- removed the 74175 at (220.8, 70.8)
- removed 74367 (x4), 7475 (x3), 7483 (x2), 75157: DIP-16_W7.62mm_vintage, Dazzler:DIP-16_W7.62mm_vintage
- removed the 7474 at (152.1, 45.6)
- removed the 7474 at (220.8, 96.1)
- removed the 7493 at (175.0, 70.8)
- removed the 7493 at (129.1, 70.8)
- removed the 7493 at (106.2, 70.8)
- removed the 74LS04 at (220.7, 121.4)
- removed the 74LS04 at (197.8, 121.4)
- removed the 74LS04 at (246.3, 96.1)
- removed the 74LS04 at (106.1, 96.1)
- removed the 74LS04 at (83.4, 96.1)
- removed the G*** at (148.0, 90.2) (x2)
- removed the H1 at (26.7, 27.9)
- removed H2: Ejector, mals-library-pcb:s100-ejector
- removed J1, J2, J3, J4, J5 (x2), J6 (x2), J7 (x2): DIP-pad, Dazzler:DIP-pad
- removed NO IC: DIP-16_W7.62mm_vintage, Dazzler:DIP-16_W7.62mm_vintage
- removed the REF** at (96.1, 88.3)
- removed the REF** at (111.3, 88.3)
- removed the REF** at (108.8, 101.0)
- removed the REF** at (98.6, 88.4)
- removed the REF** at (111.3, 100.9)
- removed the REF** at (116.4, 100.9)
- removed the REF** at (113.8, 88.2)
- removed the REF** at (121.4, 88.3)
- removed the REF** at (116.4, 88.3)
- removed the REF** at (118.9, 88.2)
- removed the REF** at (108.7, 88.2)
- removed TO BOARD 1: DIP-16_W7.62mm_vintage, Dazzler:DIP-16_W7.62mm_vintage
- added .: DIP-pad, Dazzler:DIP-pad, F.Cu at (102.1, 97.2)
- added 3417: DIP-16_W7.62mm_vintage, Dazzler:DIP-16_W7.62mm_vintage, F.Cu at (174.6, 102.6)
- added 7400: DIP-14_W7.62mm_vintage, Dazzler:DIP-14_W7.62mm_vintage, F.Cu at (37.0, 128.0)
- added 7400: DIP-14_W7.62mm_vintage, Dazzler:DIP-14_W7.62mm_vintage, F.Cu at (60.0, 77.3)
- added 7400: DIP-14_W7.62mm_vintage, Dazzler:DIP-14_W7.62mm_vintage, F.Cu at (197.5, 77.4)
- added 7400: DIP-14_W7.62mm_vintage, Dazzler:DIP-14_W7.62mm_vintage, F.Cu at (174.6, 77.3)
- added 7404: DIP-14_W7.62mm_vintage, Dazzler:DIP-14_W7.62mm_vintage, F.Cu at (220.3, 128.1)
- added 7404: DIP-14_W7.62mm_vintage, Dazzler:DIP-14_W7.62mm_vintage, F.Cu at (60.1, 102.5)
- added 7408: DIP-14_W7.62mm_vintage, Dazzler:DIP-14_W7.62mm_vintage, F.Cu at (197.4, 102.6)
- added 7408: DIP-14_W7.62mm_vintage, Dazzler:DIP-14_W7.62mm_vintage, F.Cu at (128.8, 102.6)
- added 7408: DIP-14_W7.62mm_vintage, Dazzler:DIP-14_W7.62mm_vintage, F.Cu at (37.1, 77.3)
- added 7410: DIP-14_W7.62mm_vintage, Dazzler:DIP-14_W7.62mm_vintage, F.Cu at (243.3, 77.3)
- added 7410: DIP-14_W7.62mm_vintage, Dazzler:DIP-14_W7.62mm_vintage, F.Cu at (220.4, 77.3)
- added 7410: DIP-14_W7.62mm_vintage, Dazzler:DIP-14_W7.62mm_vintage, F.Cu at (37.0, 102.6)
- added 7410: DIP-14_W7.62mm_vintage, Dazzler:DIP-14_W7.62mm_vintage, F.Cu at (59.9, 51.9)
- added 74151: DIP-16_W7.62mm_vintage, Dazzler:DIP-16_W7.62mm_vintage, F.Cu at (220.3, 102.6)
- added 74157: DIP-16_W7.62mm_vintage, Dazzler:DIP-16_W7.62mm_vintage, F.Cu at (151.7, 77.4)
- added 74157: DIP-16_W7.62mm_vintage, Dazzler:DIP-16_W7.62mm_vintage, F.Cu at (174.6, 128.1)
- added 74157: DIP-16_W7.62mm_vintage, Dazzler:DIP-16_W7.62mm_vintage, F.Cu at (243.3, 102.6)
- added 74161: DIP-16_W7.62mm_vintage, Dazzler:DIP-16_W7.62mm_vintage, F.Cu at (103.3, 128.0)
- added 74161: DIP-16_W7.62mm_vintage, Dazzler:DIP-16_W7.62mm_vintage, F.Cu at (126.2, 128.0)
- added 74175: DIP-16_W7.62mm_vintage, Dazzler:DIP-16_W7.62mm_vintage, F.Cu at (197.4, 128.1)
- added 74175: DIP-16_W7.62mm_vintage, Dazzler:DIP-16_W7.62mm_vintage, F.Cu at (243.3, 115.4)
- added 7420: DIP-14_W7.62mm_vintage, Dazzler:DIP-14_W7.62mm_vintage, F.Cu at (60.0, 128.0)
- added 7420: DIP-14_W7.62mm_vintage, Dazzler:DIP-14_W7.62mm_vintage, F.Cu at (83.0, 102.6)
- added 7430: DIP-14_W7.62mm_vintage, Dazzler:DIP-14_W7.62mm_vintage, F.Cu at (128.6, 51.9)
- added 7432: DIP-14_W7.62mm_vintage, Dazzler:DIP-14_W7.62mm_vintage, F.Cu at (105.7, 102.6)
- added 7432: DIP-14_W7.62mm_vintage, Dazzler:DIP-14_W7.62mm_vintage, F.Cu at (105.7, 51.9)
- added 7473: DIP-14_W7.62mm_vintage, Dazzler:DIP-14_W7.62mm_vintage, F.Cu at (82.9, 128.1)
- added 7473: DIP-14_W7.62mm_vintage, Dazzler:DIP-14_W7.62mm_vintage, F.Cu at (82.9, 77.3)
- added 7473: DIP-14_W7.62mm_vintage, Dazzler:DIP-14_W7.62mm_vintage, F.Cu at (82.9, 51.9)
- added 7474: DIP-14_W7.62mm_vintage, Dazzler:DIP-14_W7.62mm_vintage, F.Cu at (151.6, 102.6)
- added 7474: DIP-14_W7.62mm_vintage, Dazzler:DIP-14_W7.62mm_vintage, F.Cu at (151.6, 51.9)
- added 7493: DIP-14_W7.62mm_vintage, Dazzler:DIP-14_W7.62mm_vintage, F.Cu at (105.8, 77.3)
- added 7493: DIP-14_W7.62mm_vintage, Dazzler:DIP-14_W7.62mm_vintage, F.Cu at (128.8, 77.3)
- added 74LS04: DIP-14_W7.62mm_vintage, Dazzler:DIP-14_W7.62mm_vintage, F.Cu at (174.6, 52.0)
- added 74LS75: DIP-16_W7.62mm_vintage, Dazzler:DIP-16_W7.62mm_vintage, F.Cu at (243.3, 128.0)
- added C21: DIP-pad, Dazzler:DIP-pad, F.Cu at (102.1, 104.1)
- added C8: DIP-pad, Dazzler:DIP-pad, F.Cu at (148.0, 104.0)
- added G***: LOGO, Dazzler:bd1-Overlay-bottom, F.Cu at (147.8, 90.4)
- added G***: LOGO, Dazzler:bd1-overlay-top, F.Cu at (147.8, 90.2)
- added H1: Video, mals-library-pcb:s100-ejector, F.Cu at (270.5, 39.2)
- added H1: Ejector, mals-library-pcb:s100-ejector, F.Cu at (268.1, 29.2)
- added H1: Ejector, mals-library-pcb:s100-ejector, F.Cu at (26.8, 27.9)
- added REF**: DIP-pad, Dazzler:DIP-pad, F.Cu at (147.9, 97.3)
- added TO BOARD NO 2: DIP-16_W7.62mm_vintage, Dazzler:DIP-16_W7.62mm_vintage, F.Cu at (151.7, 128.1)
- moved REF** 0.07 mm to (37.1, 60.9)
Routing:
- net (no net): track 17513.0 -> 14508.1 mm, vias 304 -> 406
Other:
- board text added: "10K"
- board text added: "15K"
- board text added: "18K"
- board text added: "2N3904"
- board text added: "2N3906"
- board text added: "36K"
- board text added: "62K"
- board text added: "7500"
- board text added: "80K"
- board text added: "9100"
- board text added: "BLUE"
- board text added: "C1"
- board text added: "C10"
- board text added: "C11"
- board text added: "C12"
- board text added: "C13"
- board text added: "C14"
- board text added: "C18"
- board text added: "C19"
- board text added: "C22"
- board text added: "C23"
- board text added: "C24"
- board text added: "C26"
- board text added: "C27"
- board text added: "C5"
- board text added: "C9"
- board text added: "CROMEMCO DAZZLER"
- board text added: "D1"
- board text added: "D2"
- board text added: "G1"
- board text added: "Q1"
- board text added: "Q2"
- board text added: "Q3"
- board text added: "R1"
- board text added: "R18"
- board text added: "R19"
- board text added: "R2"
- board text added: "R20"
- board text added: "R21"
- board text added: "R22"
- board text added: "R23"
- board text added: "R25"
- board text added: "R26"
- board text added: "R27"
- board text added: "R28"
- board text added: "TM"
- board text removed: "C28"
- board text removed: "C29"
- board text removed: "C30"
- board text removed: "C31"
- board text removed: "C32"
- board text removed: "C33"
- board text removed: "C34"
- board text removed: "C35"
- board text removed: "C36"
- board text removed: "C37"
- board text removed: "C38"
- board text removed: "C39"
